File: 68030-RAM-IDE-V02.brd (EAGLE design)
At the start: 70 x 100 mm, 71 parts, among them IC1 REG1117, IC10 ICS570B, IC2 74HCT245PW, IC3 74AC16245, IC4 AM29F010S, IC5 74ALVT16543, IC6 74ALVT16543, IC7 XC95288XL-TQ144, IC8 K4S56163, IC9 K4S56163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

Commit message: Board not saved
Parts:
- added C37, C38: 100pF, rcl:C0603K
Connections:
- net GND: now also C37.2, C38.2
- net LE_30_RAM: now also C38.1
- net LE_RAM_30: now also C37.1
Routing:
- net GND: track 17.9 -> 22.4 mm, vias 73 -> 74
- net LE_RAM_30: track 59.3 -> 62.7 mm
- net LE_30_RAM: track 57.5 -> 60.3 mm
Changed lines of the file:
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@@
 <param name="mlMinCreamFrame" value="0mil"/>
 <param name="mlMaxCreamFrame" value="0mil"/>
-<param name="mlViaStopLimit" value="0mil"/>
+<param name="mlViaStopLimit" value="16mil"/>
 <param name="srRoundness" value="0"/>
 <param name="srMinRoundness" value="0mil"/>
@@
 <element name="R13" library="rcl" package="R0603" value="" x="49.2125" y="79.53375"/>
 <element name="SJ2" library="jumper" package="SJ_2" value="" x="51.435" y="71.27875"/>
+<element name="C37" library="rcl" package="C0603K" value="100pF" x="27.305" y="11.27125"/>
+<element name="C38" library="rcl" package="C0603K" value="100pF" x="14.44625" y="10.63625" rot="R270"/>
 </elements>
 <signals>
@@
 <via x="25.87625" y="25.87625" extent="1-16" drill="0.3"/>
 <via x="26.82875" y="25.87625" extent="1-16" drill="0.3"/>
+<contactref element="C37" pad="2"/>
+<contactref element="C38" pad="2"/>
+<wire x1="14.44625" y1="9.76125" x2="13.575" y2="8.89" width="0.254" layer="1"/>
+<wire x1="13.575" y1="8.89" x2="11.43" y2="8.89" width="0.254" layer="1"/>
+<wire x1="11.43" y1="8.89" x2="10.63625" y2="8.09625" width="0.254" layer="1"/>
+<via x="10.63625" y="8.09625" extent="1-16" drill="0.3"/>
+<wire x1="18.4404" y1="8.6106" x2="14.44625" y2="9.76125" width="0" layer="19" extent="1-1"/>
 </signal>
 <signal name="CIIN">
@@
 <contactref element="IC3" pad="26"/>
 <contactref element="IC6" pad="24"/>
-<wire x1="8.89" y1="8.89" x2="9.8044" y2="8.89" width="0.254" layer="1"/>
-<wire x1="9.8044" y1="8.89" x2="15.2262" y2="14.3118" width="0.254" layer="1"/>
-<wire x1="15.2262" y1="14.3118" x2="16.2974" y2="14.3118" width="0.254" layer="1"/>
+<wire x1="8.89" y1="8.89" x2="9.4869" y2="8.89" width="0.254" layer="1"/>
+<wire x1="9.4869" y1="8.89" x2="14.9087" y2="14.3118" width="0.254" layer="1"/>
+<wire x1="14.9087" y1="14.3118" x2="16.2974" y2="14.3118" width="0.254" layer="1"/>
 <via x="52.07" y="8.89" extent="1-16" drill="0.3"/>
 <wire x1="52.07" y1="8.89" x2="8.89" y2="8.89" width="0.254" layer="16"/>
@@
 <wire x1="29.5275" y1="47.14875" x2="30.38875" y2="48.01" width="0.254" layer="1"/>
 <wire x1="30.38875" y1="48.01" x2="30.38875" y2="56.56" width="0.254" layer="1"/>
+<contactref element="C37" pad="1"/>
+<wire x1="26.43" y1="11.27125" x2="26.43" y2="12.305" width="0.254" layer="1"/>
+<wire x1="26.43" y1="12.305" x2="25.9231" y2="12.8119" width="0.254" layer="1"/>
+<wire x1="25.9231" y1="12.8119" x2="24.3426" y2="12.8119" width="0.254" layer="1"/>
 </signal>
 <signal name="OE_30_RAM">
@@
 <wire x1="25.87625" y1="50.64125" x2="26.38875" y2="51.15375" width="0.254" layer="1"/>
 <wire x1="26.38875" y1="51.15375" x2="26.38875" y2="56.56" width="0.254" layer="1"/>
+<contactref element="C38" pad="1"/>
+<wire x1="16.2974" y1="12.7882" x2="14.85195" y2="12.7882" width="0.254" layer="1"/>
+<wire x1="14.85195" y1="12.7882" x2="14.44625" y2="12.3825" width="0.254" layer="1"/>
+<wire x1="14.44625" y1="12.3825" x2="14.44625" y2="11.51125" width="0.254" layer="1"/>
 </signal>
 <signal name="ROM_B0">
