File: 68030-RAM-IDE-V02.brd (EAGLE design)
At the start: 70 x 100 mm, 73 parts, among them IC1 REG1117, IC10 ICS570B, IC2 74HCT245PW, IC3 74AC16245, IC4 AM29F010S, IC5 74ALVT16543, IC6 74ALVT16543, IC7 XC95288XL-TQ144, IC8 K4S56163, IC9 K4S56163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

Commit message: Fixed some values in pcb and cleaned code
Parts:
- C36: value (none) -> 100nF
- R2: value 4.7 -> 4k7
Changed lines of the file:
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@@
 </element>
 <element name="C2" library="rcl" package="C0805K" value="47µF" x="30.48" y="6.35"/>
-<element name="R2" library="rcl" package="R0603" value="4.7" x="65.24625" y="29.62275" rot="R270"/>
+<element name="R2" library="rcl" package="R0603" value="4k7" x="65.24625" y="29.62275" rot="R270"/>
 <element name="R3" library="rcl" package="R2512" value="500mA" x="58.26125" y="75.72375" rot="R90"/>
 <element name="IC4" library="am29-memory" package="PLCC-SR32" value="AM29F010S" x="27.305" y="90.17" rot="R90"/>
@@
 </element>
 <element name="SJ1" library="jumper" package="SJ_2" value="" x="44.92625" y="79.85125"/>
-<element name="C36" library="rcl" package="C0603K" value="" x="45.24375" y="76.04125" rot="R270"/>
+<element name="C36" library="rcl" package="C0603K" value="100nF" x="45.24375" y="76.04125" rot="R270"/>
 <element name="R10" library="rcl" package="R0603" value="33" x="55.08625" y="75.72375" rot="R270"/>
 <element name="R11" library="rcl" package="R0603" value="33" x="52.22875" y="79.53375" rot="R180"/>
